Commit message: added arm95 in moveit config

File: arm95_description/resource/urdf/arm95.urdf (robot description, URDF)
Before this commit: robot arm95, 7 links, 6 joints
Links:
- link Link3: geometry collision mesh filename=package://arm95_description/resource/meshes/visual/Link3.stl scale=1.00000 1.00000 1.00000; visual mesh filename=package://arm95_description/resource/meshes/visual/Link3.stl scale=1.00000 1.00000 1.00000
- link Link6: geometry collision mesh filename=package://arm95_description/resource/meshes/visual/Link6.stl scale=1.00000 1.00000 1.00000; visual mesh filename=package://arm95_description/resource/meshes/visual/Link6.stl scale=1.00000 1.00000 1.00000
Joints:
- joint Joint1: axis 0.00000 0.00000 1.00000 -> 0.00000 0.00000 -1.00000; child Link1_link -> Link1
- joint Joint2: child Link2_link -> Link2; parent Link1_link -> Link1
- joint Joint3: child Link3_link -> Link3; parent Link2_link -> Link2
- joint Joint4: child Link4_link -> Link4; parent Link3_link -> Link3
- joint Joint5: axis 0.00000 0.00000 1.00000 -> 0.00000 0.00000 -1.00000; child Link5_link -> Link5; parent Link4_link -> Link4
- joint Joint6: child Tool_link -> Link6; parent Link5_link -> Link5

File: moveit_config/urdf/mcx.ros2_control.xacro (robot description, xacro)
@@ -7,5 +7,5 @@
                 <param name="robot_ip">${robot_ip}</param>
             </hardware>
-        <joint name="pr15_shoulder_pan_joint">
+        <joint name="Joint1">
             <state_interface name="position"/>
             <state_interface name="velocity"/>
@@ -13,5 +13,5 @@
             <param name="initial_position">0.0</param>
         </joint>
-        <joint name="pr15_shoulder_lift_joint">
+        <joint name="Joint2">
             <state_interface name="position"/>
             <state_interface name="velocity"/>
@@ -19,5 +19,5 @@
             <param name="initial_position">0.0</param>
         </joint>
-        <joint name="pr15_elbow_joint">
+        <joint name="Joint3">
             <state_interface name="position"/>
             <state_interface name="velocity"/>
@@ -25,5 +25,5 @@
             <param name="initial_position">0.0</param>
         </joint>
-        <joint name="pr15_wrist1_joint">
+        <joint name="Joint4">
             <state_interface name="position"/>
             <state_interface name="velocity"/>
@@ -31,5 +31,5 @@
             <param name="initial_position">0.0</param>
         </joint>
-        <joint name="pr15_wrist2_joint">
+        <joint name="Joint5">
             <state_interface name="position"/>
             <state_interface name="velocity"/>
@@ -37,5 +37,5 @@
             <param name="initial_position">0.0</param>
         </joint>
-        <joint name="pr15_wrist3_joint">
+        <joint name="Joint6">
             <state_interface name="position"/>
             <state_interface name="velocity"/>

File: moveit_config/urdf/moveit_description.urdf.xacro (robot description, xacro)
@@ -2,5 +2,5 @@
 <robot name="mcx_robot" xmlns:xacro="http://ros.org/wiki/xacro">
   <xacro:arg name="robot_ip" default="192.168.2.100"/>
-  <xacro:include filename="$(find manipulator_description)/resource/urdf/pr15.urdf"/>
+  <xacro:include filename="$(find arm95_description)/resource/urdf/arm95.urdf"/>
   <xacro:include filename="mcx.ros2_control.xacro"/>
   <xacro:mcx_ros2_control robot_ip="$(arg robot_ip)"/>

Commit message: changed joints limit

File: arm95_description/resource/urdf/arm95.urdf (robot description, URDF)
Before this commit: robot arm95, 7 links, 6 joints
Joints:
- joint Joint1: limit lower=-6.37000 upper=6.37000 effort=143.00000 velocity=3.14000 -> lower=-3.14 upper=3.14 effort=143.00000 velocity=3.14000
- joint Joint2: limit lower=-6.37000 upper=6.37000 effort=143.00000 velocity=3.14000 -> lower=-3.14 upper=3.14 effort=143.00000 velocity=3.14000
- joint Joint3: limit lower=-6.37000 upper=6.37000 effort=110.00000 velocity=3.14000 -> lower=-3.14 upper=3.14 effort=110.00000 velocity=3.14000
- joint Joint4: limit lower=-6.37000 upper=6.37000 effort=70.00000 velocity=3.14000 -> lower=-3.14 upper=3.14 effort=70.00000 velocity=3.14000
- joint Joint5: limit lower=-6.37000 upper=6.37000 effort=70.00000 velocity=3.14000 -> lower=-3.14 upper=3.14 effort=70.00000 velocity=3.14000
- joint Joint6: limit lower=-6.37000 upper=6.37000 effort=70.00000 velocity=3.14000 -> lower=-3.14 upper=3.14 effort=70.00000 velocity=3.14000
