Commit message: fixed urdf

File: arm1650_description/resource/urdf/arm1650.urdf (robot description, URDF)
Before this commit: robot arm1650, 9 links, 8 joints
Links:
- removed link arm1650_base_link
- removed link arm1650_forearm_link
- removed link arm1650_shoulder_link
- removed link arm1650_upperarm_link
- removed link arm1650_wrist1_link
- removed link arm1650_wrist2_link
- removed link arm1650_wrist3_link
- added link Base_link, mass 4.021; collision mesh filename=package://arm1650_description/resource/meshes/collision/bas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 scale=1.0 1.0 1.0; visual mesh filename=package://arm1650_description/resource/meshes/visual/base_l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 scale=1.0 1.0 1.0
- added link Link1, mass 3.661; collision mesh filename=package://arm1650_description/resource/meshes/collision/sho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 scale=1.0 1.0 1.0; visual mesh filename=package://arm1650_description/resource/meshes/visual/should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 scale=1.0 1.0 1.0
- added link Link2, mass 8.341; collision mesh filename=package://arm1650_description/resource/meshes/collision/upp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 scale=1.0 1.0 1.0; visual mesh filename=package://arm1650_description/resource/meshes/visual/uppera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 scale=1.0 1.0 1.0
- added link Link3, mass 2.311; collision mesh filename=package://arm1650_description/resource/meshes/collision/for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 scale=1.0 1.0 1.0; visual mesh filename=package://arm1650_description/resource/meshes/visual/forear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 scale=1.0 1.0 1.0
- added link Link4, mass 1.291; collision mesh filename=package://arm1650_description/resource/meshes/collision/wri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 scale=1.0 1.0 1.0; visual mesh filename=package://arm1650_description/resource/meshes/visual/wrist1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 scale=1.0 1.0 1.0
- added link Link5, mass 1.291; collision mesh filename=package://arm1650_description/resource/meshes/collision/wri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 scale=1.0 1.0 1.0; visual mesh filename=package://arm1650_description/resource/meshes/visual/wrist2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 scale=1.0 1.0 1.0
- added link Link6, mass 0.001; visual mesh filename=package://arm1650_description/resource/meshes/visual/wrist3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 scale=1.0 1.0 1.0
Joints:
- removed joint arm1650_elbow_joint
- removed joint arm1650_shoulder_lift_joint
- removed joint arm1650_shoulder_pan_joint
- removed joint arm1650_wrist1_joint
- removed joint arm1650_wrist2_joint
- removed joint arm1650_wrist3_joint
- added joint Joint1: type revolute, parent Base_link, child Link1, origin xyz=0 0 0 rpy=0 0 0, axis 0 0 1.0, limit lower=-3.14 upper=3.14 effort=0 velocity=0
- added joint Joint2: type revolute, parent Link1, child Link2, origin xyz=0 0 0.190 rpy=-1.5708 0 0, axis 0 0 1.0, limit lower=-3.14 upper=3.14 effort=0 velocity=0
- added joint Joint3: type revolute, parent Link2, child Link3, origin xyz=0 -0.8 0 rpy=0 0 0, axis 0 0 1.0, limit lower=-3.14 upper=3.14 effort=0 velocity=0
- added joint Joint4: type revolute, parent Link3, child Link4, origin xyz=0 -0.72 0 rpy=0 0 0, axis 0 0 1.0, limit lower=-3.14 upper=3.14 effort=0 velocity=0
- added joint Joint5: type revolute, parent Link4, child Link5, origin xyz=0 0 -0.191 rpy=1.5708 0 0, axis 0 0 1.0, limit lower=-3.14 upper=3.14 effort=0 velocity=0
- added joint Joint6: type revolute, parent Link5, child Link6, origin xyz=0 -0.069 0.130 rpy=0 0 0, axis 0 1.0 0, limit lower=-3.14 upper=3.14 effort=0 velocity=0
- joint tool_frame: parent arm1650_wrist3_link -> Link6
- joint world_fixed: child arm1650_base_link -> Base_link

Commit message: fixed collision model

File: arm1650_description/resource/urdf/arm1650.urdf (robot description, URDF)
Before this commit: robot arm1650, 9 links, 8 joints
Links:
- link Base_link: geometry collision mesh filename=package://arm1650_description/resource/meshes/collision/Bas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 scale=1.0 1.0 1.0; visual mesh filename=package://arm1650_description/resource/meshes/visual/base_l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 scale=1.0 1.0 1.0
- link Link1: geometry collision mesh filename=package://arm1650_description/resource/meshes/collision/Lin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 scale=1.0 1.0 1.0; visual mesh filename=package://arm1650_description/resource/meshes/visual/should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 scale=1.0 1.0 1.0
- link Link2: geometry collision mesh filename=package://arm1650_description/resource/meshes/collision/Lin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 scale=1.0 1.0 1.0; visual mesh filename=package://arm1650_description/resource/meshes/visual/uppera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 scale=1.0 1.0 1.0
- link Link3: geometry collision mesh filename=package://arm1650_description/resource/meshes/collision/Lin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 scale=1.0 1.0 1.0; visual mesh filename=package://arm1650_description/resource/meshes/visual/forear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 scale=1.0 1.0 1.0
- link Link4: geometry collision mesh filename=package://arm1650_description/resource/meshes/collision/Lin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 scale=1.0 1.0 1.0; visual mesh filename=package://arm1650_description/resource/meshes/visual/wrist1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 scale=1.0 1.0 1.0
- link Link5: geometry collision mesh filename=package://arm1650_description/resource/meshes/collision/Lin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 scale=1.0 1.0 1.0; visual mesh filename=package://arm1650_description/resource/meshes/visual/wrist2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 scale=1.0 1.0 1.0
- link Link6: geometry collision mesh filename=package://arm1650_description/resource/meshes/collision/Lin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 scale=1.0 1.0 1.0; visual mesh filename=package://arm1650_description/resource/meshes/visual/wrist3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 scale=1.0 1.0 1.0

Commit message: fixed joint limits

File: arm1650_description/resource/urdf/arm1650.urdf (robot description, URDF)
Before this commit: robot arm1650, 9 links, 8 joints
Joints:
- joint Joint1: limit lower=-3.14 upper=3.14 effort=0 velocity=0 -> lower=-3.14 upper=3.14 effort=0 velocity=1.745329251994
- joint Joint2: limit lower=-3.14 upper=3.14 effort=0 velocity=0 -> lower=-3.14 upper=3.14 effort=0 velocity=1.745329251994
- joint Joint3: limit lower=-3.14 upper=3.14 effort=0 velocity=0 -> lower=-3.14 upper=3.14 effort=0 velocity=2.617993877992
- joint Joint4: limit lower=-3.14 upper=3.14 effort=0 velocity=0 -> lower=-3.14 upper=3.14 effort=0 velocity=2.617993877992
- joint Joint5: limit lower=-3.14 upper=3.14 effort=0 velocity=0 -> lower=-3.14 upper=3.14 effort=0 velocity=2.617993877992
- joint Joint6: limit lower=-3.14 upper=3.14 effort=0 velocity=0 -> lower=-3.14 upper=3.14 effort=0 velocity=2.617993877992
